File: tool-power-supply-v1/bus12v.kicad_sch (KiCad schematic)
At the start: 37 parts, among them J3 DB128V-5.08-2P-GN-S, J4 DB128V-5.08-2P-GN-S, J5 XT60PW-F (ESC power), J6 Fan (1 GND, 2 +12V, 3 TACH, 4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, Q1 AO4407C P-FET, Q2 2N7002, Q3 AO4407C P-FET, Q4 2N7002, Q5 AO4407C P-FET, Q6 2N7002, U3 INA226AIDGSR

Commit message: schematic update: cleaned up by using sheet labels and busses, updated documentation
Co-Authored-By: Claude Sonnet 5.5 <noreply@anthropic.com>
Connections:
- net 12V_A_FUSED: no longer names the net of F3.2, Q1.1 (S), Q1.2 (S), Q1.3 (S), R7.1, XH1.3, XH1.4
- net 12V_A_GATE: no longer names the net of Q1.4 (G), Q2.3 (D), R7.2
- net 12V_A_OUT: no longer names the net of J3.1 (Pin_1), Q1.5 (D), Q1.6 (D), Q1.7 (D), Q1.8 (D), R9.1
- net 12V_B_FUSED: no longer names the net of F4.2, Q3.1 (S), Q3.2 (S), Q3.3 (S), R11.1, XH2.3, XH2.4
- net 12V_B_GATE: no longer names the net of Q3.4 (G), Q4.3 (D), R11.2
- net 12V_B_OUT: no longer names the net of J4.1 (Pin_1), Q3.5 (D), Q3.6 (D), Q3.7 (D), Q3.8 (D), R13.1
- net EN_12V_A renamed EN.12V_A
- net EN_12V_B renamed EN.12V_B
- net EN_ESC renamed EN.ESC
- net ESC_FUSED: no longer names the net of F5.2, Q5.1 (S), Q5.2 (S), Q5.3 (S), R15.1, XH3.3, XH3.4
- net ESC_GATE: no longer names the net of Q5.4 (G), Q6.3 (D), R15.2
- net ESC_OUT: no longer names the net of J5.1 (Pin_1), Q5.5 (D), Q5.6 (D), Q5.7 (D), Q5.8 (D), R17.1
- net FAN_12V: no longer names the net of F6.2, J6.2 (Pin_2)
- net FAN_PWM renamed FAN.PWM
- net FAN_TACH renamed FAN.TACH
- net I2C_SCL renamed I2C.SCL
- net I2C_SDA renamed I2C.SDA
- net INA_ALERT renamed I2C.ALERT
- net LED12_A: no longer names the net of D4.2 (A), R6.2
- net SENSE_12V_A renamed SENSE.12V_A
- net SENSE_12V_B renamed SENSE.12V_B
- net SENSE_ESC renamed SENSE.ESC
Other:
- note added: "100 uF"
- note added: "12V_A: fuse, P-FET switch, presence sense"
- note added: "12V_B: fuse, P-FET switch, presence sense"
- note added: "5 mohm shunt: Kelvin-connect INA pins at the pads"
- note added: "Bus protection, bulk capacitance, rail LED"
- note added: "ESC: fuse, P-FET switch, presence sense"
- note added: "LED"
- note added: "TVS SMCJ15A"
- note removed: "12 V tap A (3 A blade fuse, P-FET switch, presence sense)"
- note removed: "12 V tap B (3 A blade fuse, P-FET switch, presence sense)"
- note removed: "Bus protection, bulk capacitance and rail LED"
- note removed: "ESC branch (7.5 A blade fuse, P-FET switch, presence sense)"
