File: tool-power-supply-v1/bus12v.kicad_sch (KiCad schematic)
At the start: 37 parts, among them J3 DB128V-5.08-2P-GN-S, J4 DB128V-5.08-2P-GN-S, J5 XT60PW-F (ESC power), J6 Fan (1 GND, 2 +12V, 3 TACH, 4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, Q1 AO4407C P-FET, Q2 2N7002, Q3 AO4407C P-FET, Q4 2N7002, Q5 AO4407C P-FET, Q6 2N7002, U3 INA226AIDGSR

Commit message: schematic update: finished cleaning up
Parts:
- removed C3: 100nF 50V X7R, Capacitor_SMD:C_0603_1608Metric, symbol Device:C
- removed C4: 100uF 35V, Capacitor_SMD:CP_Elec_6.3x7.7, symbol Device:C_Polarized
- removed F3, F4: 3A ATO blade fuse, symbol Device:Fuse
- removed F5: 7.5A ATO blade fuse, symbol Device:Fuse
- removed F6: PTC 500mA hold 33V, Fuse:Fuse_1206_3216Metric, symbol Device:Polyfuse
- removed J3: DB128V-5.08-2P-GN-S, TerminalBlock_CUI:TerminalBlock_CUI_TB007-508-02_1x02_P5.08mm_Horizontal, symbol Connector:Screw_Terminal_01x02
- removed J5: XT60PW-F (ESC power), Connector_AMASS:AMASS_XT60PW-F_1x02_P7.20mm_Horizontal, symbol Connector_Generic:Conn_01x02
- removed J6: Fan (1 GND, 2 +12V, 3 TACH, 4 PWM), Connector_Molex:Molex_KK-254_AE-6410-04A_1x04_P2.54mm_Vertical, symbol Connector_Generic:Conn_01x04
- removed Q2: 2N7002, Package_TO_SOT_SMD:SOT-23, symbol Transistor_FET:2N7002
- removed Q5: AO4407C P-FET, Package_SO:SOIC-8_3.9x4.9mm_P1.27mm, symbol Transistor_FET:FDS9435A
- removed R10, R11, R12, R14, R15, R16, R18, R19, R7, R8: 10k (1%), Resistor_SMD:R_0603_1608Metric, symbol Device:R
- removed R13, R17, R9: 33k (1%), Resistor_SMD:R_0603_1608Metric, symbol Device:R
- removed R5: 5mR 2512 (shunt), Resistor_SMD:R_2512_6332Metric, symbol Device:R
- removed R6: 4.7k (1%), Resistor_SMD:R_0603_1608Metric, symbol Device:R
- removed XH1: Keystone 3557 blade holder 12V_A, HF_Footprints:355720, symbol HF_Passives:3557-20
- removed XH2: Keystone 3557 blade holder 12V_B, HF_Footprints:355720, symbol HF_Passives:3557-20
- removed XH3: Keystone 3557 blade holder ESC, HF_Footprints:355720, symbol HF_Passives:3557-20
- added C3: 100uF, Capacitor_SMD:CP_Elec_6.3x7.7, symbol Device:C_Polarized_Small
- added C4: 100nF, Capacitor_SMD:C_0603_1608Metric, symbol Device:C_Small
- added F3: 500mA, Fuse:Fuse_1206_3216Metric, symbol Device:Polyfuse_Small
- added F4, F5: 3A, HF_Footprints:Fuse_Blade_Keystone_3557-20_P13.47mm, symbol HF_Passives:Fuse_Blade_Keystone_3557
- added F6: 7.5A, HF_Footprints:Fuse_Blade_Keystone_3557-20_P13.47mm, symbol HF_Passives:Fuse_Blade_Keystone_3557
- added J3: Fan (1 GND, 2 +12V, 3 TACH, 4 PWM), Connector_Molex:Molex_KK-254_AE-6410-04A_1x04_P2.54mm_Vertical, symbol Connector_Generic:Conn_01x04
- added J5: DB128V-5.08-2P-GN-S, TerminalBlock_CUI:TerminalBlock_CUI_TB007-508-02_1x02_P5.08mm_Horizontal, symbol Connector:Screw_Terminal_01x02
- added J6: XT60PW-F, Connector_AMASS:AMASS_XT60PW-F_1x02_P7.20mm_Horizontal, symbol Connector_Generic:Conn_01x02
- added Q2: AO4407C, Package_SO:SOIC-8_3.9x4.9mm_P1.27mm, symbol Transistor_FET:FDS9435A
- added Q5: 2N7002, Package_TO_SOT_SMD:SOT-23, symbol Transistor_FET:2N7002
- added R10, R12, R8: 33k, Resistor_SMD:R_0603_1608Metric, symbol Device:R_Small_US
- added R11, R13, R14, R15, R16, R17, R18, R19, R6, R9: 10k, Resistor_SMD:R_0603_1608Metric, symbol Device:R_Small_US
- added R5: 5m, Resistor_SMD:R_2512_6332Metric, symbol Device:R_Small_US
- added R7: 4.7k, Resistor_SMD:R_0603_1608Metric, symbol Device:R_Small_US
- D3: value SMCJ15A TVS -> SMCJ15A; Function (none) -> SMCJ15A TVS
- D4: value LED yellow -> NCD0603Y2; Color (none) -> yellow
- Q1, Q3: value AO4407C P-FET -> AO4407C; Function (none) -> AO4407C P-FET
Connections:
- net 12V_BUS: now also C3.1, F3.1, F4.1, F5.1, F6.1, R5.2, R7.1
- net 12V_MOD: now also R5.1
- net 3V3_BUCK: now also R14.2, R15.2, R16.2
- net 3V3_MCU: now also C4.1, R6.2
- net EN.12V_A: now also Q4.1 (G), R14.1
- net EN.12V_B: now also Q5.1 (G), R15.1; no longer Q4.1 (G)
- net EN.ESC: now also R16.1
- net FAN.PWM: now also J3.4 (Pin_4)
- net FAN.TACH: now also J3.3 (Pin_3), R6.1
- net GND: now also C3.2, C4.2, J3.1 (Pin_1), J5.2 (Pin_2), J6.2 (Pin_2), Q5.2 (S), R11.2, R13.2, R9.2
- net SENSE.12V_A: now also R8.2, R9.1
- net SENSE.12V_B: now also R10.2, R11.1
- net SENSE.ESC: now also R12.2, R13.1
- net at Q3.5 (D), Q3.6 (D), Q3.7 (D)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: now also J6.1 (Pin_1), R12.1; no longer J4.1 (Pin_1)
- net at Q6.3 (D): now also Q3.4 (G), R19.2
- net at Q4.3 (D): now also Q1.4 (G), R17.2; no longer Q3.4 (G)
- net at D4.2 (A): now also R7.2
- net at Q1.1 (S), Q1.2 (S), Q1.3 (S): now also F4.2, R17.1
- net at Q1.5 (D), Q1.6 (D), Q1.7 (D)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: now also J4.1 (Pin_1), R8.1
- net at Q3.1 (S), Q3.2 (S), Q3.3 (S): now also F6.2, R19.1
- new net: F5.2, Q2.1 (S), Q2.2 (S), Q2.3 (S), R18.1
- new net: Q2.4 (G), Q5.3 (D), R18.2
- new net: J5.1 (Pin_1), Q2.5 (D), Q2.6 (D), Q2.7 (D), Q2.8 (D), R10.1
- new net: F3.2, J3.2 (Pin_2)
Other:
- note added: "R5 5 mR, dV = I x R at the module output current: idle 0.08 A: 0.4 mV spin coater 5.9 A: 29.5 mV module limit 6.7 A: 33.5 mV (7.37 A for 10 s: 36.9 mV) INA226 shunt range +-81.92 mV = 16.4 A"
- note removed: "100 uF"
- note removed: "LED"
- note removed: "TVS SMCJ15A"

Commit message: layout update: finished cleanup
Parts:
- removed J6: XT60PW-F, Connector_AMASS:AMASS_XT60PW-F_1x02_P7.20mm_Horizontal, symbol Connector_Generic:Conn_01x02
- added J6: XT60PB-F, HF_Footprints:XT60PBF, symbol HF_Connectors:XT60PB-F
Connections:
- net GND: now also J6.2 (-)
- net at Q3.5 (D), Q3.6 (D), Q3.7 (D)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: now also J6.1 (+)
- net 3V3_BUCK renamed 3V3_RAIL
Changed lines of the file:
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@@
 	)
 	(symbol
+		(lib_id "HF_Connectors:XT60PB-F")
+		(at 187.96 163.83 180)
+		(unit 1)
+		(body_style 1)
+		(exclude_from_sim no)
+		(in_bom yes)
+		(on_board yes)
+		(in_pos_files yes)
+		(dnp no)
+		(property "Reference" "J6"
+			(at 160.02 162.052 0)
+			(show_name no)
+			(do_not_autoplace no)
+			(effects
+				(font
+					(size 1.27 1.27)
+				)
+				(justify right)
+			)
+		)
+		(property "Value" "XT60PB-F"
+			(at 160.02 164.592 0)
+			(show_name no)
+			(do_not_autoplace no)
+			(effects
+				(font
+					(size 1.27 1.27)
+				)
+				(justify right)
+			)
+		)
+		(property "Footprint" "HF_Footprints:XT60PBF"
+			(at 187.96 163.83 0)
+			(hide yes)
+			(show_name no)
+			(do_not_autoplace no)
+			(effects
+				(font
+					(size 1.27 1.27)
+				)
+			)
+		)
+		(property "Datasheet" "https://www.tme.eu/Document/aa7a0328674fda4109d00dc748bb5162/XT60UPB-F.pdf"
+			(at 187.96 163.83 0)
+			(hide yes)
+			(show_name no)
+			(do_not_autoplace no)
+			(effects
+				(font
+					(size 1.27 1.27)
+				)
+			)
+		)
+		(property "Description" "XT60PB-F vertical female, ESC power (the ESC lead is male)"
+			(at 187.96 163.83 0)
+			(hide yes)
+			(show_name no)
+			(do_not_autoplace no)
+			(effects
+				(font
+					(size 1.27 1.27)
+				)
+			)
+		)
+		(property "LCSC" "C19268038"
+			(at 187.96 163.83 0)
+			(hide yes)
+			(show_name no)
+			(do_not_autoplace no)
+			(effects
+				(font
+					(size 1.27 1.27)
+				)
+			)
+		)
+		(property "MPN" "XT60PB-F"
+			(at 187.96 163.83 0)
+			(hide yes)
+			(show_name no)
+			(do_not_autoplace no)
+			(effects
+				(font
+					(size 1.27 1.27)
+				)
+			)
+		)
+		(property "Manufacturer" "AMASS"
+			(at 187.96 163.83 0)
+			(hide yes)
+			(show_name no)
+			(do_not_autoplace no)
+			(effects
+				(font
+					(size 1.27 1.27)
+				)
+			)
+		)
+		(pin "1"
+		)
+		(pin "2"
+		)
+		(instances
+			(project "tool-power-supply-v1"
+				(path "/38374745-796d-4ac0-8538-65a2602e3d35/0cb51aae-028b-431a-91a3-4936dff542ce"
+					(reference "J6")
+					(unit 1)
+				)
+			)
+		)
+	)
+	(symbol
 		(lib_id "power:+3V3")
 		(at 213.36 163.83 0)
@@
 			)
 		)
-		(property "Value" "3V3_BUCK"
+		(property "Value" "3V3_RAIL"
 			(at 208.534 159.258 0)
 			(show_name no)
@@
 	)
 	(symbol
-		(lib_id "Connector_Generic:Conn_01x02")
-		(at 182.88 161.29 0)
-		(mirror y)
-		(unit 1)
-		(body_style 1)
-		(exclude_from_sim no)
-		(in_bom yes)
-		(on_board yes)
-		(in_pos_files yes)
-		(dnp no)
-		(property "Reference" "J6"
-			(at 182.88 157.988 0)
-			(show_name no)
-			(do_not_autoplace no)
-			(effects
-				(font
-					(size 1.27 1.27)
-				)
-			)
-		)
-		(property "Value" "XT60PW-F"
-			(at 177.546 176.082 0)
-			(hide yes)
-			(show_name no)
-			(do_not_autoplace no)
-			(effects
-				(font
-					(size 1.27 1.27)
-				)
-			)
-		)
-		(property "Footprint" "Connector_AMASS:AMASS_XT60PW-F_1x02_P7.20mm_Horizontal"
-			(at 182.88 161.29 0)
-			(hide yes)
-			(show_name no)
-			(do_not_autoplace no)
-			(effects
-				(font
-					(size 1.27 1.27)
-				)
-			)
-		)
-		(property "Datasheet" ""
-			(at 182.88 161.29 0)
-			(hide yes)
-			(show_name no)
-			(do_not_autoplace no)
-			(effects
-				(font
-					(size 1.27 1.27)
-				)
-			)
-		)
-		(property "Description" "XT60PW-F female, ESC power (the ESC lead is male)"
-			(at 182.88 161.29 0)
-			(hide yes)
-			(show_name no)
-			(do_not_autoplace no)
-			(effects
-				(font
-					(size 1.27 1.27)
-				)
-			)
-		)
-		(property "LCSC" "C428722"
-			(at 182.88 161.29 0)
-			(hide yes)
-			(show_name no)
-			(do_not_autoplace no)
-			(effects
-				(font
-					(size 1.27 1.27)
-				)
-			)
-		)
-		(property "MPN" "XT60PW-F"
-			(at 182.88 161.29 0)
-			(hide yes)
-			(show_name no)
-			(do_not_autoplace no)
-			(effects
-				(font
-					(size 1.27 1.27)
-				)
-			)
-		)
-		(property "Manufacturer" "AMASS"
-			(at 182.88 161.29 0)
-			(hide yes)
-			(show_name no)
-			(do_not_autoplace no)
-			(effects
-				(font
-					(size 1.27 1.27)
-				)
-			)
-		)
-		(pin "1"
-		)
-		(pin "2"
-		)
-		(instances
-			(project "tool-power-supply-v1"
-				(path "/38374745-796d-4ac0-8538-65a2602e3d35/0cb51aae-028b-431a-91a3-4936dff542ce"
-					(reference "J6")
-					(unit 1)
-				)
-			)
-		)
-	)
-	(symbol
 		(lib_id "Device:R_Small_US")
 		(at 193.04 165.1 0)
@@
 			)
 		)
-		(property "Value" "3V3_BUCK"
+		(property "Value" "3V3_RAIL"
 			(at 208.534 48.768 0)
 			(show_name no)
@@
 			)
 		)
-		(property "Value" "3V3_BUCK"
+		(property "Value" "3V3_RAIL"
 			(at 208.534 103.378 0)
 			(show_name no)
