File: tool-power-supply-v1/rails.kicad_sch (KiCad schematic)
At the start: 48 parts, among them J10 DB128V-5.08-2P-GN-S, J7 DB128V-5.08-2P-GN-S, J8 DB128V-5.08-2P-GN-S, J9 DB128V-5.08-2P-GN-S, U10 TPS2553DBVR, U11 TPS2553DBVR, U4 AP63205WU-7, U5 INA226AIDGSR, U6 TPS2553DBVR, U7 TPS2553DBVR, U8 AP63203WU-7, U9 INA226AIDGSR

Commit message: schematic update: cleaned up by using sheet labels and busses, updated documentation
Co-Authored-By: Claude Sonnet 5.5 <noreply@anthropic.com>
Connections:
- net 3V3_A_OUT renamed SENSE.3V3_A
- net 3V3_B_OUT renamed SENSE.3V3_B
- net 5V_A_OUT: no longer names the net of J7.1 (Pin_1), R24.1, U6.6 (OUT)
- net 5V_BUCK: no longer names the net of C7.1, C8.1, L1.2, R20.1, U4.1 (FB), U5.10 (Vin+)
- net 5V_B_OUT: no longer names the net of J8.1 (Pin_1), R28.1, U7.6 (OUT)
- net BST_3V3: no longer names the net of C13.1, U8.6 (BST)
- net BST_5V: no longer names the net of C6.1, U4.6 (BST)
- net EN_3V3_A renamed EN.3V3_A
- net EN_3V3_B renamed EN.3V3_B
- net EN_5V_A renamed EN.5V_A
- net EN_5V_B renamed EN.5V_B
- net FAULT_3V3 renamed FAULT.3V3
- net FAULT_5V renamed FAULT.5V
- net I2C_SCL renamed I2C.SCL
- net I2C_SDA renamed I2C.SDA
- net ILIM_3V3_A: no longer names the net of R32.1, U10.5 (ILIM)
- net ILIM_3V3_B: no longer names the net of R35.1, U11.5 (ILIM)
- net ILIM_5V_A: no longer names the net of R22.1, U6.5 (ILIM)
- net ILIM_5V_B: no longer names the net of R26.1, U7.5 (ILIM)
- net INA_ALERT renamed I2C.ALERT
- net LED3_A: no longer names the net of D6.2 (A), R31.2
- net LED5_A: no longer names the net of D5.2 (A), R21.2
- net SENSE_5V_A renamed SENSE.5V_A
- net SENSE_5V_B renamed SENSE.5V_B
- net SW_3V3: no longer names the net of C13.2, L2.1, U8.5 (SW)
- net SW_5V: no longer names the net of C6.2, L1.1, U4.5 (SW)
Other:
- note added: "3.3 V monitor (INA226 #3, address 0x42) and rail LED"
- note added: "3.3 V taps A and B (TPS2553, enable pull-up; the tap net is the presence sense)"
- note added: "5 V monitor (INA226 #2, address 0x41) and rail LED"
- note added: "5 V taps A and B (TPS2553, enable pull-up, presence sense)"
- note removed: "3.3 V monitor (INA226 #3, 0x42) and rail LED"
- note removed: "3.3 V taps A and B (TPS2553, enable control; tap net is the sense input)"
- note removed: "5 V monitor (INA226 #2, 0x41) and rail LED"
- note removed: "5 V taps A and B (TPS2553, enable control, presence sense)"
