File: tool-power-supply-v1/rails.kicad_sch (KiCad schematic)
At the start: 48 parts, among them J10 DB128V-5.08-2P-GN-S, J7 DB128V-5.08-2P-GN-S, J8 DB128V-5.08-2P-GN-S, J9 DB128V-5.08-2P-GN-S, U10 TPS2553DBVR, U11 TPS2553DBVR, U4 AP63205WU-7, U5 INA226AIDGSR, U6 TPS2553DBVR, U7 TPS2553DBVR, U8 AP63203WU-7, U9 INA226AIDGSR

Commit message: schematic update: finished cleaning up
Parts:
- removed C10, C11, C16, C17, C18, C9: 100nF 50V X7R, Capacitor_SMD:C_0603_1608Metric, symbol Device:C
- removed C12, C5: 10uF 50V, Capacitor_SMD:C_1206_3216Metric, symbol Device:C
- removed C13, C6: 100nF 50V, Capacitor_SMD:C_0603_1608Metric, symbol Device:C
- removed C14, C15, C7, C8: 22uF 25V, Capacitor_SMD:C_0805_2012Metric, symbol Device:C
- removed L1, L2: 4.7uH, Inductor_SMD:L_Sumida_CDMC6D28_7.25x6.5mm, symbol Device:L
- removed R20, R30: 33mR 1206 (shunt), Resistor_SMD:R_1206_3216Metric, symbol Device:R
- removed R21: 1.5k (1%), Resistor_SMD:R_0603_1608Metric, symbol Device:R
- removed R22, R26, R32, R35: 33k (1%), Resistor_SMD:R_0603_1608Metric, symbol Device:R
- removed R23, R25, R27, R29, R33, R34, R36, R37: 10k (1%), Resistor_SMD:R_0603_1608Metric, symbol Device:R
- removed R24, R28: 4.7k (1%), Resistor_SMD:R_0603_1608Metric, symbol Device:R
- removed R31: 680 (1%), Resistor_SMD:R_0603_1608Metric, symbol Device:R
- removed U5, U9: INA226AIDGSR, Package_SO:MSOP-10_3x3mm_P0.5mm, symbol Sensor_Energy:INA226
- removed U6, U7: TPS2553DBVR, HF_Footprints:SOT95P280X145-6N, symbol HF_ICs:TPS2553DBVR
- removed U8: AP63203WU-7, Package_TO_SOT_SMD:TSOT-23-6, symbol Regulator_Switching:AP63203WU
- added C10, C11, C12, C9: 22uF, Capacitor_SMD:C_0805_2012Metric, symbol Device:C_Small
- added C13, C14, C15, C16, C17, C18, C7, C8: 100nF, Capacitor_SMD:C_0603_1608Metric, symbol Device:C_Small
- added C5, C6: 10uF, Capacitor_SMD:C_1206_3216Metric, symbol Device:C_Small
- added L1, L2: 4.7uH, Inductor_SMD:L_Sumida_CDMC6D28_7.25x6.5mm, symbol Device:L_Small
- added R20: 1.5k, Resistor_SMD:R_0603_1608Metric, symbol Device:R_Small_US
- added R21: 680, Resistor_SMD:R_0603_1608Metric, symbol Device:R_Small_US
- added R22, R23: 33m, Resistor_SMD:R_1206_3216Metric, symbol Device:R_Small_US
- added R24, R25, R26, R27, R33, R35, R36, R37: 10k, Resistor_SMD:R_0603_1608Metric, symbol Device:R_Small_US
- added R28, R29, R30, R31: 33k, Resistor_SMD:R_0603_1608Metric, symbol Device:R_Small_US
- added R32, R34: 4.7k, Resistor_SMD:R_0603_1608Metric, symbol Device:R_Small_US
- added U5: AP63203WU-7, Package_TO_SOT_SMD:TSOT-23-6, symbol Regulator_Switching:AP63203WU
- added U6, U7: INA226AIDGSR, Package_SO:MSOP-10_3x3mm_P0.5mm, symbol Sensor_Energy:INA226
- added U8, U9: TPS2553DBVR, HF_Footprints:SOT95P280X145-6N, symbol HF_ICs:TPS2553DBVR
- D5, D6: value LED yellow -> NCD0603Y2; Color (none) -> yellow
Connections:
- net 12V_BUS: now also C5.1, C6.1, U5.2 (EN), U5.3 (IN)
- net 3V3_BUCK: now also C10.1, C12.1, L2.2, R23.1, R24.2, R25.2, R26.2, R27.2, U5.1 (FB), U7.10 (Vin+)
- net 3V3_MCU: now also C13.1, C14.1, U6.2 (A0), U6.6 (VS), U7.6 (VS)
- net 3V3_RAIL: now also C17.1, C18.1, R21.1, R23.2, U7.8 (Vbus), U7.9 (Vin-)
- net 5V_RAIL: now also C15.1, C16.1, R20.1, R22.2, U6.8 (Vbus), U6.9 (Vin-), U8.1 (IN), U9.1 (IN)
- net EN.3V3_A: now also R26.1
- net EN.3V3_B: now also R27.1
- net EN.5V_A: now also R24.1, U8.3 (EN)
- net EN.5V_B: now also R25.1, U9.3 (EN)
- net FAULT.5V: now also U8.4 (~{FAULT}), U9.4 (~{FAULT})
- net GND: now also C10.2, C11.2, C12.2, C13.2, C14.2, C15.2, C16.2, C17.2, C18.2, C5.2, C6.2, C9.2, R28.2, R29.2, R30.2, R31.2, R33.2, R35.2, R36.2, R37.2, U5.4 (GND), U6.1 (A1), U6.7 (GND), U7.1 (A1), U7.7 (GND), U8.2 (GND), U9.2 (GND)
- net I2C.ALERT: now also U6.3 (~{Alert}), U7.3 (~{Alert})
- net I2C.SCL: now also U6.5 (SCL), U7.5 (SCL)
- net I2C.SDA: now also U6.4 (SDA), U7.2 (A0), U7.4 (SDA)
- net SENSE.3V3_A: now also J7.1 (Pin_1), R36.1; no longer J9.1 (Pin_1)
- net SENSE.3V3_B: now also J8.1 (Pin_1), R37.1; no longer J10.1 (Pin_1)
- net SENSE.5V_A: now also R32.2, R33.1
- net SENSE.5V_B: now also R34.2, R35.1
- net at U11.5 (ILIM): now also R31.1
- net at D6.2 (A): now also R21.2
- net at U4.1 (FB): now also C11.1, C9.1, L1.2, R22.1, U6.10 (Vin+)
- net at U4.6 (BST): now also C7.1
- net at U4.5 (SW): now also C7.2, L1.1
- net at D5.2 (A): now also R20.2
- net at U10.5 (ILIM): now also R30.1
- new net: R29.1, U9.5 (ILIM)
- new net: J10.1 (Pin_1), R34.1, U9.6 (OUT)
- new net: R28.1, U8.5 (ILIM)
- new net: J9.1 (Pin_1), R32.1, U8.6 (OUT)
- new net: C8.2, L2.1, U5.5 (SW)
- new net: C8.1, U5.6 (BST)
Other:
- note added: "(there is a gen rule for inductor selection based on ripple)"
- note added: "L1 Isat 9.0 A (20% drop), Irms 5.5 A, DCR 38 mOhm max 5 V at 2 A: ripple about 0.56 A pk-pk at 1.1 MHz, peak about 2.3 A AP63205 high-side limit 3.1 A max, so Isat has 2.9x margin R20 33 mR, dV = I x R at the 5 V rail current: idle 0.04 A: 1.3 mV spin coater 1.04 A: 34.3 mV all taps at peak 1.13 A: 37.3 mV all taps at current limit 1.85 A: 61.0 mV (2 A buck limit: 66 mV) INA226 shunt range +-81.9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"

Commit message: layout update: finished cleanup
Parts:
- removed J9: DB128V-5.08-2P-GN-S, TerminalBlock_CUI:TerminalBlock_CUI_TB007-508-02_1x02_P5.08mm_Horizontal, symbol Connector:Screw_Terminal_01x02
- renumbered J10 to J9
Connections:
- net 3V3_RAIL: now also R24.2, R25.2, R26.2, R27.2
- net 5V_LINK: now reaches R32.1, U8.6 (OUT)
- net 3V3_BUCK: no longer names the net of C10.1, C12.1, L2.2, R23.1, U5.1 (FB), U7.10 (Vin+)
- net 3V3_BUCK: no longer R24.2, R25.2, R26.2, R27.2
