File: tool-power-supply-v1/mains.kicad_sch (KiCad schematic)
At the start: 26 parts, among them J1 AC IN (L, N, PE), J2 AC OUT (L, N, PE), U1 IRM-90-12, U2 ACS712ELCTR-20A-T

Commit message: schematic update: finished cleaning up
Parts:
- removed C1, C2: 100nF 50V X7R, Capacitor_SMD:C_0603_1608Metric, symbol Device:C
- removed F1: 3A Slo-Blo 3AG, symbol Device:Fuse
- removed F2: 10A ceramic fast-blow 3AG 250VAC, symbol Device:Fuse
- removed R1, R2, R3, R4: 33k (1%), Resistor_SMD:R_0603_1608Metric, symbol Device:R
- removed XF1: 01020074Z clip F1 in, HF_Footprints:01020074Z, symbol HF_Passives:01020074Z
- removed XF2: 01020074Z clip F1 out, HF_Footprints:01020074Z, symbol HF_Passives:01020074Z
- removed XF3: 01020074Z clip F2 in, HF_Footprints:01020074Z, symbol HF_Passives:01020074Z
- removed XF4: 01020074Z clip F2 out, HF_Footprints:01020074Z, symbol HF_Passives:01020074Z
- added C1, C2: 100nF, Capacitor_SMD:C_0603_1608Metric, symbol Device:C_Small
- added F1: 10A, HF_Footprints:Fuse_3AG_6.3x32mm_Clips_Littelfuse_102_122_P34.21mm, symbol HF_Passives:Fuse_3AG_6.3x32mm
- added F2: 3A, HF_Footprints:Fuse_3AG_6.3x32mm_Clips_Littelfuse_102_122_P34.21mm, symbol HF_Passives:Fuse_3AG_6.3x32mm
- added R1, R2, R3, R4: 33k, Resistor_SMD:R_0603_1608Metric, symbol Device:R_Small_US
- D1: value LED red -> KT-0603R; Color (none) -> red
- D2: value 1N4148W (LED antiparallel) -> 1N4148W; Function (none) -> 1N4148W (LED antiparallel)
- RV1: value 14D241K MOV -> 14D241K; Function (none) -> MOV, line to neutral after the fuse side of the module bran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
- SJ1: value PE tie (PE-GND) -> CHASSIS-PE
- SJ2: value CHASSIS-PE -> CHASSIS-GND
- SJ3: value CHASSIS-GND -> PE tie (PE-GND)
Connections:
- net 5V_RAIL: now also C1.1
- net GND: now also SJ2.2 (B), C1.2, C2.2; no longer SJ1.2 (B)
- net at H1.1, H2.1, H3.1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: now also SJ1.1 (A); no longer SJ3.1 (A)
- net at J1.1: now also F1.1, F2.1, R1.1
- net at U2.1 (IP+), U2.2 (IP+): now also F1.2
- net at RV1.1, U1.AC_L (AC/L): now also F2.2
- net at J1.3, J2.3: now also SJ1.2 (B), SJ3.1 (A); no longer SJ1.1 (A), SJ2.2 (B)
- net at U2.6 (FILTER): now also C2.1
- net at D1.2 (A), D2.1 (K): now also R4.2
- new net: R3.2, R4.1
- new net: R2.2, R3.1
- new net: R1.2, R2.1
Other:
- note added: "4 x 33k = 132k across 120 VAC (170 V peak) I rms 0.91 mA: 0.11 W total, 27 mW per resistor (0603 is 0.1 W) 42 V peak per resistor (0603 about 75 V working, verify) LED half-wave: I peak 1.3 mA, average 0.4 mA, 0.8 mW"
- note added: "FILTER 100 nF: f(-3 dB) about 0.9 to 1.2 kHz 1/(2 pi x 1.7k x 100n) = 0.94 kHz with the typical internal RF of 1.7k; the datasheet rise time for 100 nF (291 us) gives 1.2 kHz"
- note removed: "FILTER 100 nF (about 940 Hz)"
- note removed: "MOV"
- note removed: "PE tie"
- note removed: "clips for F1"
- note removed: "clips for F2"

Commit message: layout update: doing some reorg before routing, locking in prog before adding CAN + expander.
Parts:
- H1, H2, H3, H4: value M3 hole -> M2 hole; footprint MountingHole:MountingHole_3.2mm_M3_Pad -> MountingHole:MountingHole_2.2mm_M2_Pad
- RV1: value 14D241K -> 10D241K; footprint Varistor:RV_Disc_D16.5mm_W6.7mm_P7.5mm -> Varistor:RV_Disc_D12mm_W5.4mm_P7.5mm; LCSC C49072887 -> C49072899; MPN 14D241K -> 10D241K; Note Verify disc size against datasheet -> Verify disc size and thickness against the C49072899 datash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
Connections:
- net at J1.3, J2.3, SJ3.1 (A): no longer SJ1.2 (B)
- new net: SJ1.1 (A), SJ2.1 (A)
- now unconnected: H1.1, H2.1, H3.1, H4.1
- no-connect marks 0 -> 5
Other:
- note added: "CHASSIS?"
- note removed: "CHASSIS"
Changed lines of the file:
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@@
 		)
 	)
-	(text "CHASSIS"
+	(text "CHASSIS?"
 		(exclude_from_sim no)
-		(at 86.614 215.392 0)
+		(at 115.824 214.376 0)
 		(effects
 			(font
@@
 	)
 	(junction
-		(at 144.78 185.42)
-		(diameter 0)
-		(color 0 0 0 0)
-	)
-	(junction
-		(at 88.9 210.82)
-		(diameter 0)
-		(color 0 0 0 0)
-	)
-	(junction
 		(at 254 43.18)
 		(diameter 0)
@@
 	)
 	(junction
-		(at 134.62 210.82)
-		(diameter 0)
-		(color 0 0 0 0)
-	)
-	(junction
-		(at 101.6 210.82)
-		(diameter 0)
-		(color 0 0 0 0)
-	)
-	(junction
 		(at 162.56 185.42)
 		(diameter 0)
@@
 	)
 	(junction
-		(at 76.2 210.82)
-		(diameter 0)
-		(color 0 0 0 0)
-	)
-	(junction
 		(at 76.2 156.21)
 		(diameter 0)
 		(color 0 0 0 0)
 	)
+	(no_connect
+		(at 76.2 210.82)
+	)
+	(no_connect
+		(at 101.6 210.82)
+	)
+	(no_connect
+		(at 144.78 210.82)
+	)
+	(no_connect
+		(at 88.9 210.82)
+	)
+	(no_connect
+		(at 63.5 210.82)
+	)
 	(wire
 		(pts
@@
 	(wire
 		(pts
-			(xy 144.78 210.82) (xy 144.78 185.42)
-		)
-		(stroke
-			(width 0)
-			(type default)
-		)
-	)
-	(wire
-		(pts
 			(xy 134.62 210.82) (xy 134.62 223.52)
 		)
@@
 	(wire
 		(pts
-			(xy 63.5 210.82) (xy 134.62 210.82)
-		)
-		(stroke
-			(width 0)
-			(type default)
-		)
-	)
-	(wire
-		(pts
 			(xy 254 43.18) (xy 269.24 43.18)
 		)
@@
 			)
 		)
-		(property "Value" "M3 hole"
+		(property "Value" "M2 hole"
 			(at 68.072 208.34 0)
 			(show_name no)
@@
 			)
 		)
-		(property "Footprint" "MountingHole:MountingHole_3.2mm_M3_Pad"
+		(property "Footprint" "MountingHole:MountingHole_2.2mm_M2_Pad"
 			(at 63.5 203.2 0)
 			(hide yes)
@@
 		(exclude_from_sim no)
 		(in_bom yes)
-		(on_board yes)
+		(on_board no)
 		(in_pos_files yes)
 		(dnp no)
@@
 			)
 		)
-		(property "Value" "M3 hole"
+		(property "Value" "M2 hole"
 			(at 81.026 208.34 0)
 			(show_name no)
@@
 			)
 		)
-		(property "Footprint" "MountingHole:MountingHole_3.2mm_M3_Pad"
+		(property "Footprint" "MountingHole:MountingHole_2.2mm_M2_Pad"
 			(at 76.2 203.2 0)
 			(hide yes)
@@
 		(exclude_from_sim no)
 		(in_bom yes)
-		(on_board yes)
+		(on_board no)
 		(in_pos_files yes)
 		(dnp no)
@@
 			)
 		)
-		(property "Value" "14D241K"
+		(property "Value" "10D241K"
 			(at 164.49 141.3 0)
 			(show_name no)
@@
 			)
 		)
-		(property "Footprint" "Varistor:RV_Disc_D16.5mm_W6.7mm_P7.5mm"
+		(property "Footprint" "Varistor:RV_Disc_D12mm_W5.4mm_P7.5mm"
 			(at 161.29 139.7 0)
 			(hide yes)
@@
 			)
 		)
-		(property "LCSC" "C49072887"
+		(property "LCSC" "C49072899"
 			(at 161.29 139.7 0)
 			(hide yes)
@@
 			)
 		)
-		(property "MPN" "14D241K"
+		(property "MPN" "10D241K"
 			(at 161.29 139.7 0)
 			(hide yes)
@@
 			)
 		)
-		(property "Note" "Verify disc size against datasheet"
+		(property "Note" "Verify disc size and thickness against the C49072899 datasheet; footprint is the 12 mm disc, 5.4 mm thick"
 			(at 161.29 139.7 0)
 			(hide yes)
@@
 			)
 		)
-		(property "Value" "M3 hole"
+		(property "Value" "M2 hole"
 			(at 93.726 208.534 0)
 			(show_name no)
@@
 			)
 		)
-		(property "Footprint" "MountingHole:MountingHole_3.2mm_M3_Pad"
+		(property "Footprint" "MountingHole:MountingHole_2.2mm_M2_Pad"
 			(at 88.9 203.2 0)
 			(hide yes)
@@
 			)
 		)
-		(property "Value" "M3 hole"
+		(property "Value" "M2 hole"
 			(at 106.68 208.594 0)
 			(show_name no)
@@
 			)
 		)
-		(property "Footprint" "MountingHole:MountingHole_3.2mm_M3_Pad"
+		(property "Footprint" "MountingHole:MountingHole_2.2mm_M2_Pad"
 			(at 101.6 203.2 0)
 			(hide yes)

Commit message: layout update: finished cleanup
Parts:
- H1, H2, H3, H4: value M2 hole -> M3 hole; footprint MountingHole:MountingHole_2.2mm_M2_Pad -> MountingHole:MountingHole_3.2mm_M3_Pad_Via
Connections:
- net LIVE: now reaches F1.1, F2.1, J1.1, R1.1
- net NEUTRAL: now reaches D1.1 (K), D2.2 (A), J1.2, J2.2, RV1.2, U1.AC_N (AC/N)
- net PE: now reaches J1.3, J2.3, SJ3.1 (A)
Other:
- note removed: "L"
- note removed: "N"
- note removed: "PE"
Changed lines of the file:
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@@
 		)
 	)
-	(text "N"
-		(exclude_from_sim no)
-		(at 66.04 171.45 0)
-		(effects
-			(font
-				(size 1.27 1.27)
-			)
-			(justify left bottom)
-		)
-	)
 	(text "4 x 33k = 132k across 120 VAC (170 V peak)\nI rms 0.91 mA: 0.11 W total, 27 mW per resistor (0603 is 0.1 W)\n42 V peak per resistor (0603 about 75 V working, verify)\nLED half-wave: I peak 1.3 mA, average 0.4 mA, 0.8 mW"
 		(exclude_from_sim no)
@@
 		)
 	)
-	(text "PE"
-		(exclude_from_sim no)
-		(at 60.96 184.15 0)
-		(effects
-			(font
-				(size 1.27 1.27)
-			)
-			(justify left bottom)
-		)
-	)
 	(text "Module branch: 3 A time-lag 3AG, surge protection, IRM-90-12"
 		(exclude_from_sim no)
@@
 		)
 	)
-	(text "L"
-		(exclude_from_sim no)
-		(at 55.88 57.15 0)
-		(effects
-			(font
-				(size 1.27 1.27)
-			)
-			(justify left bottom)
-		)
-	)
 	(text "CHASSIS?"
 		(exclude_from_sim no)
@@
 		)
 	)
+	(label "NEUTRAL"
+		(at 52.07 60.96 0)
+		(effects
+			(font
+				(size 1.27 1.27)
+			)
+			(justify left bottom)
+		)
+	)
+	(label "PE"
+		(at 52.07 63.5 0)
+		(effects
+			(font
+				(size 1.27 1.27)
+			)
+			(justify left bottom)
+		)
+	)
+	(label "LIVE"
+		(at 52.07 58.42 0)
+		(effects
+			(font
+				(size 1.27 1.27)
+			)
+			(justify left bottom)
+		)
+	)
 	(hierarchical_label "ACS_OUT"
 		(shape output)
@@
 			)
 		)
-		(property "Value" "M2 hole"
+		(property "Value" "M3 hole"
 			(at 68.072 208.34 0)
 			(show_name no)
@@
 			)
 		)
-		(property "Footprint" "MountingHole:MountingHole_2.2mm_M2_Pad"
+		(property "Footprint" "MountingHole:MountingHole_3.2mm_M3_Pad_Via"
 			(at 63.5 203.2 0)
 			(hide yes)
@@
 			)
 		)
-		(property "Value" "M2 hole"
+		(property "Value" "M3 hole"
 			(at 81.026 208.34 0)
 			(show_name no)
@@
 			)
 		)
-		(property "Footprint" "MountingHole:MountingHole_2.2mm_M2_Pad"
+		(property "Footprint" "MountingHole:MountingHole_3.2mm_M3_Pad_Via"
 			(at 76.2 203.2 0)
 			(hide yes)
@@
 			)
 		)
-		(property "Value" "M2 hole"
+		(property "Value" "M3 hole"
 			(at 93.726 208.534 0)
 			(show_name no)
@@
 			)
 		)
-		(property "Footprint" "MountingHole:MountingHole_2.2mm_M2_Pad"
+		(property "Footprint" "MountingHole:MountingHole_3.2mm_M3_Pad_Via"
 			(at 88.9 203.2 0)
 			(hide yes)
@@
 			)
 		)
-		(property "Value" "M2 hole"
+		(property "Value" "M3 hole"
 			(at 106.68 208.594 0)
 			(show_name no)
@@
 			)
 		)
-		(property "Footprint" "MountingHole:MountingHole_2.2mm_M2_Pad"
+		(property "Footprint" "MountingHole:MountingHole_3.2mm_M3_Pad_Via"
 			(at 101.6 203.2 0)
 			(hide yes)
