File: tool-power-supply-v1/tool-power-supply-v1.kicad_sch (KiCad schematic)
At the start: 0 parts

Commit message: schematic update: finished cleaning up
Other:
- note added: "AC ISO"
- note removed: "12 V bus and branch switches"
- note removed: "5 V / 3.3 V rails and taps"
- note removed: "Mains zone"
- note removed: "Pico 2, analog inputs, SSR drive"
- note removed: "Rev 1 power board. Sheets connect through sheet pins; control signals travel on the bus groups EN, SENSE, FAULT, I2C and FAN. Source of truth for decisions: design-context/design-decisions.md; BOM: design-context/bom.md; pin map: design-context/pin-map.md. Generated by tools/schematic/build2.py."

Commit message: layout update: finished cleanup
Other:
- sheet mcu ports: added 5V_LINK; removed none
- sheet rails ports: added 5V_LINK; removed none
Changed lines of the file:
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@@
+		)
+	)
+	(wire
+		(pts
+			(xy 173.99 149.86) (xy 232.41 149.86)
+		)
+		(stroke
+			(width 0)
+			(type default)
 		)
 	)
@@
 	(wire
 		(pts
+			(xy 232.41 96.52) (xy 275.59 96.52)
+		)
+		(stroke
+			(width 0)
+			(type default)
+		)
+	)
+	(wire
+		(pts
 			(xy 105.41 55.88) (xy 105.41 69.85)
+		)
+		(stroke
+			(width 0)
+			(type default)
+		)
+	)
+	(wire
+		(pts
+			(xy 232.41 149.86) (xy 232.41 96.52)
 		)
 		(stroke
@@
 			)
 		)
+		(pin "5V_LINK" input
+			(at 275.59 96.52 180)
+			(effects
+				(font
+					(size 1.27 1.27)
+				)
+				(justify left)
+			)
+		)
 		(instances
 			(project "tool-power-supply-v1"
@@
 			(effects
 				(font
+					(size 1.27 1.27)
+				)
+				(justify right)
+			)
+		)
+		(pin "5V_LINK" output
+			(at 173.99 149.86 0)
+			(effects
+				(font
