File: tool-power-supply-v1/mcu.kicad_sch (KiCad schematic)
At the start: 16 parts, among them J11 DB128V-5.08-2P-GN-S, J12 DB128V-5.08-2P-GN-S, Q7 2N7002 (SSR drive), U12 Raspberry Pi Pico 2

Commit message: schematic update: finished cleaning up
Parts:
- removed R38, R39, R40, R45: 4.7k (1%), Resistor_SMD:R_0603_1608Metric, symbol Device:R
- removed R41, R42, R43: 10k (1%), Resistor_SMD:R_0603_1608Metric, symbol Device:R
- removed R44: 1k (1%), Resistor_SMD:R_0603_1608Metric, symbol Device:R
- added R38, R39, R41, R43: 4.7k, Resistor_SMD:R_0603_1608Metric, symbol Device:R_Small_US
- added R40: 1k, Resistor_SMD:R_0603_1608Metric, symbol Device:R_Small_US
- added R42, R44, R45: 10k, Resistor_SMD:R_0603_1608Metric, symbol Device:R_Small_US
- D7: value SS14 (5V to VSYS) -> SS14; Function (none) -> SS14 (5V to VSYS)
- Q7: value 2N7002 (SSR drive) -> 2N7002; Function (none) -> 2N7002 (SSR drive)
- TH1: value NTC 10k (module) -> 10k; Type (none) -> NTC thermistor, on the module
- U12: value Raspberry Pi Pico 2 -> SC1631; Function (none) -> Raspberry Pi Pico 2; MPN SC1631 (Pico 2) -> SC1631
Connections:
- net 3V3_MCU: now also R38.2, R39.2, R44.1, R45.1
- net ACS_OUT: now also R43.1
- net GND: now also R41.2, R42.2
- net I2C.SCL: now also R38.1
- net I2C.SDA: now also R39.1
- net at SJ4.3 (B), U12.24 (GPIO18): now also R40.1
- net at Q7.1 (G): now also R40.2, R41.1
- net at J11.1 (Pin_1), U12.34 (GPIO28_ADC2): now also R45.2
- net at TH1.1, U12.32 (GPIO27_ADC1): now also R44.2
- net at U12.31 (GPIO26_ADC0): now also R42.1, R43.2

Commit message: layout update: finished cleanup
Parts:
- added C19, C20: 100nF, Capacitor_SMD:C_0603_1608Metric, symbol Device:C_Small
- added J10: DB128V-5.08-4P-GN-S, TerminalBlock_CUI:TerminalBlock_CUI_TB007-508-04_1x04_P5.08mm_Horizontal, symbol Connector:Screw_Terminal_01x04
- added R40: 10k, Resistor_SMD:R_0603_1608Metric, symbol Device:R_Small_US
- added R41: 120, Resistor_SMD:R_0603_1608Metric, symbol Device:R_Small_US
- added SJ4: SJ CAN term, Jumper:SolderJumper-2_P1.3mm_Bridged_RoundedPad1.0x1.5mm, symbol Jumper:SolderJumper_2_Bridged
- added U12: TCA9534PWR, Package_SO:TSSOP-16_4.4x5mm_P0.65mm, symbol Interface_Expansion:TCA9534
- added U14: SN65HVD230DR, Package_SO:SOIC-8_3.9x4.9mm_P1.27mm, symbol Interface_CAN_LIN:SN65HVD230
- renumbered R40 to R42, R41 to R43, R42 to R44, R43 to R45, R44 to R46, R45 to R47, SJ4 to SJ5, SJ5 to SJ6, U12 to U13
Connections:
- net 3V3_MCU: now also C19.1, C20.1, U12.16 (VDD), U14.3 (VCC)
- net GND: now also C19.2, C20.2, J10.3 (Pin_3), R40.2, U12.1 (A0), U12.2 (A1), U12.3 (A2), U12.8 (GND), U14.2 (GND)
- net I2C.SCL: now also U12.14 (SCL)
- net I2C.SDA: now also U12.15 (SDA)
- net SENSE.12V_A: now also U12.4 (P0); no longer U13.20 (GPIO15)
- net SENSE.12V_B: now also U12.5 (P1); no longer U13.27 (GPIO21)
- net SENSE.3V3_A: now also U12.10 (P5); no longer U13.4 (GPIO2)
- net SENSE.3V3_B: now also U12.11 (P6); no longer U13.5 (GPIO3)
- net SENSE.5V_A: now also U12.7 (P3); no longer U13.1 (GPIO0)
- net SENSE.5V_B: now also U12.9 (P4); no longer U13.2 (GPIO1)
- net SENSE.ESC: now also U12.6 (P2); no longer U13.29 (GPIO22)
- new net: J10.4 (Pin_4), SJ4.1 (A), U14.6 (CANL)
- new net: R41.1, SJ4.2 (B)
- new net: J10.2 (Pin_2), R41.2, U14.7 (CANH)
- new net: R40.1, U14.8 (Rs)
- new net 5V_LINK: J10.1 (Pin_1)
- new net CAN_RX: U13.2 (GPIO1), U14.4 (R)
- new net CAN_TX: U13.1 (GPIO0), U14.1 (D)
- no-connect marks 5 -> 13
Other:
- note added: "CAN: can2040 on GP0 (TX) and GP1 (RX); SJ6 = 120R termination"
- note added: "Control board link: 5 V (from 5 V tap A), CANH, GND, CANL"
- note added: "I2C expander (PCA9535C, 0x20): the 7 tap-sense inputs; 9 spare pins"

Commit message: layout update: finished routing
Connections:
- net EN.12V_A: now also U13.10 (GPIO7); no longer U13.16 (GPIO12)
- net EN.12V_B: now also U13.11 (GPIO8); no longer U13.17 (GPIO13)
- net EN.3V3_A: now also U13.14 (GPIO10); no longer U13.11 (GPIO8)
- net EN.3V3_B: now also U13.19 (GPIO14); no longer U13.12 (GPIO9)
- net EN.5V_A: now also U13.4 (GPIO2); no longer U13.9 (GPIO6)
- net EN.5V_B: now also U13.12 (GPIO9); no longer U13.10 (GPIO7)
- net EN.ESC: now also U13.16 (GPIO12); no longer U13.19 (GPIO14)
- net FAN.PWM: now also U13.17 (GPIO13); no longer U13.21 (GPIO16)
- net FAN.TACH: now also U13.20 (GPIO15); no longer U13.25 (GPIO19)
- net FAULT.5V: now also U13.5 (GPIO3); no longer U13.14 (GPIO10)
- net I2C.ALERT: now also U13.9 (GPIO6); no longer U13.26 (GPIO20)
