File: tool-power-supply-v1/tool-power-supply-v1.kicad_pcb (KiCad board)
At the start: 2 copper layers, 90 x 160 mm, 118 parts, among them J1 AC IN (L, N, PE), J10 DB128V-5.08-2P-GN-S, J11 DB128V-5.08-2P-GN-S, J12 DB128V-5.08-2P-GN-S, J2 AC OUT (L, N, PE), J3 Fan (1 GND, 2 +12V, 3 TACH, 4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, J4 DB128V-5.08-2P-GN-S, J5 DB128V-5.08-2P-GN-S, J6 XT60PW-F, J7 DB128V-5.08-2P-GN-S, J8 DB128V-5.08-2P-GN-S, J9 DB128V-5.08-2P-GN-S, Q1 AO4407C, Q2 AO4407C, Q3 AO4407C, Q4 2N7002, Q5 2N7002, Q6 2N7002, Q7 2N7002, U1 IRM-90-12, U10 TPS2553DBVR, U11 TPS2553DBVR, U12 SC1631, U2 ACS712ELCTR-20A-T, U3 INA226AIDGSR, U4 AP63205WU-7, U5 AP63203WU-7, U6 INA226AIDGSR, U7 INA226AIDGSR, U8 TPS2553DBVR, U9 TPS2553DBVR

Commit message: layout update: finished cleanup
Parts:
- removed the J9 at (183.6, 143.0)
- added C19: 100nF, Capacitor_SMD:C_0603_1608Metric, F.Cu at (174.9, 65.9)
- added C20: 100nF, Capacitor_SMD:C_0603_1608Metric, F.Cu at (169.5, 118.3)
- added J10: DB128V-5.08-4P-GN-S, TerminalBlock_CUI:TerminalBlock_CUI_TB007-508-04_1x04_P5.08mm_Horizontal, F.Cu at (183.6, 131.4)
- added R40: 10k, Resistor_SMD:R_0603_1608Metric, F.Cu at (174.2, 114.7)
- added R41: 120, Resistor_SMD:R_0603_1608Metric, F.Cu at (174.0, 122.0)
- added SJ4: SJ CAN term, Jumper:SolderJumper-2_P1.3mm_Bridged_RoundedPad1.0x1.5mm, F.Cu at (174.1, 124.3)
- added U12: TCA9534PWR, Package_SO:TSSOP-16_4.4x5mm_P0.65mm, F.Cu at (177.4, 71.5)
- added U14: SN65HVD230DR, Package_SO:SOIC-8_3.9x4.9mm_P1.27mm, F.Cu at (174.1, 118.3)
- H1, H2, H3, H4: value M2 hole -> M3 hole; footprint MountingHole:MountingHole_2.2mm_M2_Pad -> MountingHole:MountingHole_3.2mm_M3_Pad_Via
- J6: value XT60PW-F -> XT60PB-F; footprint Connector_AMASS:AMASS_XT60PW-F_1x02_P7.20mm_Horizontal -> HF_Footprints:XT60PBF
- moved D4 101.4 mm to (104.4, 167.7), turned to -90 degrees
- moved R7 99.6 mm to (106.2, 167.7), turned to -90 degrees
- moved C13 75.2 mm to (159.8, 133.3), turned to 180 degrees
- moved L1 73.1 mm to (163.2, 119.2)
- moved C7 68.4 mm to (158.0, 118.5)
- moved R34 67.9 mm to (180.1, 81.3), turned to 90 degrees
- moved D7 66.0 mm to (180.0, 43.4), turned to 180 degrees
- moved U4 63.6 mm to (157.4, 121.2), turned to 0 degrees
- moved R35 63.0 mm to (180.1, 84.4), turned to 90 degrees
- moved R15 62.5 mm to (171.4, 70.2)
- moved R25 57.3 mm to (171.4, 59.8), turned to 0 degrees
- moved R24 56.8 mm to (171.4, 57.2), turned to 0 degrees
- moved R37 56.6 mm to (182.1, 84.4), turned to 90 degrees
- moved R30 51.9 mm to (175.9, 155.4), turned to 180 degrees
- moved C12 51.9 mm to (156.6, 137.8), turned to 90 degrees
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- renumbered J10 to J9, R40 to R42, R41 to R43, R42 to R44, R43 to R45, R44 to R46, R45 to R47, SJ4 to SJ5, SJ5 to SJ6, U12 to U13
Connections:
- net Net-(D1-K) renamed /mains/NEUTRAL
- net Net-(F1-Pad1) renamed /mains/LIVE
- net Net-(SJ3-A) renamed /mains/PE
- C10 pad 1: 3V3_BUCK -> Net-(U5-FB)
- C12 pad 1: 3V3_BUCK -> Net-(U5-FB)
- H1 pad 1: (no net) -> unconnected-(H1-Pad1)
- H2 pad 1: (no net) -> unconnected-(H2-Pad1)_5
- H3 pad 1: (no net) -> unconnected-(H3-Pad1)_4
- H4 pad 1: (no net) -> unconnected-(H4-Pad1)_1
- L2 pad 2: 3V3_BUCK -> Net-(U5-FB)
- R14 pad 2: 3V3_BUCK -> 3V3_RAIL
- R15 pad 2: 3V3_BUCK -> 3V3_RAIL
- R16 pad 2: 3V3_BUCK -> 3V3_RAIL
- R23 pad 1: 3V3_BUCK -> Net-(U5-FB)
- R24 pad 2: 3V3_BUCK -> 3V3_RAIL
- R25 pad 2: 3V3_BUCK -> 3V3_RAIL
- R26 pad 2: 3V3_BUCK -> 3V3_RAIL
- R27 pad 2: 3V3_BUCK -> 3V3_RAIL
- R32 pad 1: Net-(J9-Pin_1) (its old number) -> /mcu/5V_LINK
- U13 pad 1: /bus12v/SENSE.5V_A -> /mcu/CAN_TX
- U13 pad 2: /bus12v/SENSE.5V_B -> /mcu/CAN_RX
- U13 pad 20: /bus12v/SENSE.12V_A -> unconnected-(U13-GPIO15-Pad20)
- U13 pad 27: /bus12v/SENSE.12V_B -> unconnected-(U13-GPIO21-Pad27)
- U13 pad 29: /bus12v/SENSE.ESC -> unconnected-(U13-GPIO22-Pad29)
- U13 pad 4: /bus12v/SENSE.3V3_A -> unconnected-(U13-GPIO2-Pad4)
- U13 pad 5: /bus12v/SENSE.3V3_B -> unconnected-(U13-GPIO3-Pad5)
- U5 pad 1: 3V3_BUCK -> Net-(U5-FB)
- U7 pad 10: 3V3_BUCK -> Net-(U5-FB)
- U8 pad 6: Net-(J9-Pin_1) (its old number) -> /mcu/5V_LINK
Other:
- board text added: "(isolation barrier; traces only from the AC pins)"
- board text added: "12V_BUS / ESC path (about 8.3 A): wide F.Cu pour, 5 A+ min,"
- board text added: "COPPER POUR PLAN (hatched = keep out)"
- board text added: "K1 MAINS ZONE: no GND / LV pour, either layer"
- board text added: "K1 mains zone: no LV pour (3.2 mm to L/N, 1.6 mm L-N and mains-PE)"
- board text added: "K2 IRM-90-12 BODY: no pour, either layer"
- board text added: "K2 module body: no pour, window at the DC pins"
- board text added: "K3 M3 holes: floating, r 4.25 clear (7 mm washer)"
- board text added: "K3 M3 holes: no pour within r 4.25 (floating)"
- board text added: "K4"
- board text added: "K4 ACS712: pads only (isolation gap under the body)"
- board text added: "K5 L1, L2: no F.Cu pour (small SW node), B.Cu solid"
- board text added: "K6 Pico pocket (dashed, no hatch): SMD logic parts under the Pico,"
- board text added: "Pico AGND joins GND at one point at the Pico"
- board text added: "Pour (outside the keep-outs): GND on B.Cu, stitched to F.Cu GND"
- board text added: "from the module DC pins to F4-F6 and the XT60"
- board text added: "max height 7 mm (sockets 8.5 mm); no pour restriction"
- board text added: "only Mains / PE copper; 3.2 mm clear of L / N pads"
- board text added: "window: +Vo / -Vo pour allowed"
- board text added: "with vias every ~10 mm and at each bypass cap"

Commit message: layout update: finished routing
Parts:
- moved R10 25.6 mm to (158.2, 101.4)
- moved R12 25.6 mm to (160.2, 101.4)
- moved R32 25.6 mm to (162.2, 101.4)
- moved R34 25.6 mm to (164.2, 101.4)
- moved R8 25.6 mm to (156.2, 101.4)
- moved R36 24.8 mm to (167.5, 101.4), turned to 90 degrees
- moved C19 24.5 mm to (158.5, 84.1)
- moved U12 24.5 mm to (161.0, 89.7)
- moved R11 21.1 mm to (158.2, 98.3)
- moved R13 21.1 mm to (160.2, 98.3)
- moved R33 21.1 mm to (162.2, 98.3)
- moved R35 21.1 mm to (164.2, 98.3)
- moved R9 21.1 mm to (156.2, 98.3)
- moved R37 20.1 mm to (167.5, 98.3), turned to -90 degrees
- moved R27 17.7 mm to (171.4, 82.7)
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Connections:
- U13 pad 10: /bus12v/EN.5V_B -> /bus12v/EN.12V_A
- U13 pad 11: /bus12v/EN.3V3_A -> /bus12v/EN.12V_B
- U13 pad 12: /bus12v/EN.3V3_B -> /bus12v/EN.5V_B
- U13 pad 14: /mcu/FAULT.5V -> /bus12v/EN.3V3_A
- U13 pad 16: /bus12v/EN.12V_A -> /bus12v/EN.ESC
- U13 pad 17: /bus12v/EN.12V_B -> /bus12v/FAN.PWM
- U13 pad 19: /bus12v/EN.ESC -> /bus12v/EN.3V3_B
- U13 pad 20: unconnected-(U13-GPIO15-Pad20) -> /bus12v/FAN.TACH
- U13 pad 21: /bus12v/FAN.PWM -> unconnected-(U13-GPIO16-Pad21)
- U13 pad 25: /bus12v/FAN.TACH -> unconnected-(U13-GPIO19-Pad25)
- U13 pad 26: /bus12v/I2C.ALERT -> unconnected-(U13-GPIO20-Pad26)
- U13 pad 4: unconnected-(U13-GPIO2-Pad4) -> /bus12v/EN.5V_A
- U13 pad 5: unconnected-(U13-GPIO3-Pad5) -> /mcu/FAULT.5V
- U13 pad 9: /bus12v/EN.5V_A -> /bus12v/I2C.ALERT
Routing:
- net 3V3_MCU: track 0.00 -> 314.0 mm, vias 0 -> 8
- net /bus12v/I2C.SDA: track 0.00 -> 228.7 mm, vias 0 -> 4
- net /bus12v/I2C.SCL: track 0.00 -> 214.5 mm, vias 0 -> 4
- net /bus12v/I2C.ALERT: track 0.00 -> 200.3 mm, vias 0 -> 3
- net 3V3_RAIL: track 0.00 -> 181.9 mm, vias 0 -> 13
- net 12V_BUS: track 0.00 -> 163.4 mm, vias 0 -> 16
- net 5V_RAIL: track 0.00 -> 161.7 mm, vias 0 -> 8
- net /bus12v/EN.12V_A: track 0.00 -> 128.2 mm, vias 0 -> 1
- net Net-(J4-Pin_1): track 0.00 -> 125.5 mm, vias 0 -> 2
- net /mains/NEUTRAL: track 0.00 -> 123.0 mm, vias 0 -> 1
- net Net-(J5-Pin_1): track 0.00 -> 110.7 mm, vias 0 -> 2
- net /bus12v/SENSE.3V3_B: track 0.00 -> 109.8 mm, vias 0 -> 2
- net Net-(J6-+): track 0.00 -> 109.7 mm, vias 0 -> 6
- net /bus12v/EN.12V_B: track 0.00 -> 106.8 mm, vias 0 -> 1
- net /mcu/FAULT.3V3: track 0.00 -> 105.8 mm, vias 0 -> 2
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- added copper zone on B.Cu, net GND
- added copper zone on F.Cu, net GND
- added copper zone on In1.Cu, net GND
- added copper zone on In2.Cu, net GND
Other:
- copper layers 2 -> 4
- board text added: "12V_BUS / ESC path (7.5 A): outer layers only, about 3.2 mm per layer at 1 oz"
- board text added: "In2 GND 0.5 oz / B.Cu SIG+PWR 1 oz. Mains copper on F.Cu / B.Cu only."
- board text added: "K1 mains zone: no LV pour (3.2 mm to L/N, 1.6 mm L-N and mains-PE), all 4 layers"
- board text added: "K1 to K5 are also real rule areas (copper fill not allowed only)"
- board text added: "K2 module body: no pour on any layer, window at the DC pins"
- board text added: "K3 M3 holes: floating, r 4.25 clear (7 mm washer), all layers"
- board text added: "K4 ACS712: pads only (isolation gap under the body), all layers"
- board text added: "K5 L1, L2: no F.Cu pour (small SW node); In1 GND solid beneath"
- board text added: "Outer pours: GND stitched to In1 / In2 (vias every ~10 mm, at each bypass cap)"
- board text added: "Stack-up (JLC04161H-7628, 1.6 mm): F.Cu SIG+PWR 1 oz / In1 GND 0.5 oz /"
- board text added: "for a 20 C rise, so pour it on both F.Cu and B.Cu with stitching vias"
- board text added: "mains pad copper + 3.2 mm (span of each part pads); only Mains / PE copper"
- board text removed: "12V_BUS / ESC path (about 8.3 A): wide F.Cu pour, 5 A+ min,"
- board text removed: "K1 mains zone: no LV pour (3.2 mm to L/N, 1.6 mm L-N and mains-PE)"
- board text removed: "K2 module body: no pour, window at the DC pins"
- board text removed: "K3 M3 holes: floating, r 4.25 clear (7 mm washer)"
- board text removed: "K4 ACS712: pads only (isolation gap under the body)"
- board text removed: "K5 L1, L2: no F.Cu pour (small SW node), B.Cu solid"
- board text removed: "Pour (outside the keep-outs): GND on B.Cu, stitched to F.Cu GND"
- board text removed: "from the module DC pins to F4-F6 and the XT60"
- board text removed: "only Mains / PE copper; 3.2 mm clear of L / N pads"
- board text removed: "with vias every ~10 mm and at each bypass cap"
